File: hardware/control-board/control-board.kicad_sch (KiCad schematic)
At the start: 44 parts, among them J10 Conn_01x09_Socket, J11 Conn_01x09_Socket, J12 Conn_01x12_Pin, J9 Conn_01x13_Socket

Commit message: wip - first pass done
Parts:
- D1, D2, D3, D4: footprint LED_THT:LED_D3.0mm -> Eurorack Common:LED_D3.0mm; symbol Device:LED_Dual_Bidirectional -> Eurorack Common:LED_Dual_Bidirectional_3mm
- R1, R10, R11, R12, R13, R14, R15, R16, R2, R3, R4, R5, R6, R7, R8, R9: footprint Resistor_THT:R_Axial_DIN0207_L6.3mm_D2.5mm_P7.62mm_Horizontal -> Eurorack Common:R_Axial_DIN0207_L6.3mm_D2.5mm_P7.62mm_Horizontal; symbol Device:R -> Eurorack Common:R_DIN0207
Connections:
- net AUDIO_OUT_A: now reaches J13.T, R13.1
- net AUDIO_IN_B: now reaches J4.T, R6.1
- net AUDIO_IN_A: now reaches J2.T, R4.1
- net AUDIO_OUT_B: now reaches J14.T, R14.1
- net AUDIO_OUT_MIX: now reaches J16.T, R16.1
- net AUDIO_IN_C: now reaches J6.T, R9.1
- net AUDIO_OUT_C: now reaches J15.T, R15.1
- net AUDIO_IN_D: now reaches J8.T, R12.1
Other:
- moved on the sheet: R12, R13, R14, R15, R16, R4, R6, R9

Commit message: chore: clean up the boards
Parts:
- D1, D2, D3, D4: value LED_Dual_Bidirectional -> Bipolar LED
- J1, J13, J14, J15, J16, J2, J3, J4, J5, J6, J7, J8: value ~ -> Thonkicon
- J10, J11: value Conn_01x09_Socket -> 01x09 Male Pin Header
- J12: value Conn_01x12_Pin -> 01x12 Male Pin Header
- J9: value Conn_01x13_Socket -> 01x13 Male Pin Header
- RV1, RV2, RV3, RV4: value 100K -> A100K
- SW1, SW2, SW3, SW4: value ~ -> Subminiture SPDT
Changed lines of the file:
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@@
 			)
 		)
-		(property "Value" "~"
+		(property "Value" "Thonkicon"
 			(at 265.43 45.0849 0)
 			(effects
@@
 			)
 		)
-		(property "Value" "~"
+		(property "Value" "Thonkicon"
 			(at 34.29 113.6649 0)
 			(effects
@@
 			)
 		)
-		(property "Value" "Conn_01x09_Socket"
+		(property "Value" "01x09 Male Pin Header"
 			(at 158.242 33.528 0)
 			(effects
@@
 			)
 		)
-		(property "Value" "LED_Dual_Bidirectional"
+		(property "Value" "Bipolar LED"
 			(at 259.8547 25.4 0)
 			(effects
@@
 			)
 		)
-		(property "Value" "LED_Dual_Bidirectional"
+		(property "Value" "Bipolar LED"
 			(at 259.8547 57.15 0)
 			(effects
@@
 			)
 		)
-		(property "Value" "~"
+		(property "Value" "Thonkicon"
 			(at 34.29 69.2149 0)
 			(effects
@@
 			)
 		)
-		(property "Value" "LED_Dual_Bidirectional"
+		(property "Value" "Bipolar LED"
 			(at 259.8547 92.71 0)
 			(effects
@@
 			)
 		)
-		(property "Value" "Conn_01x12_Pin"
+		(property "Value" "01x12 Male Pin Header"
 			(at 209.55 32.258 0)
 			(effects
@@
 			)
 		)
-		(property "Value" "~"
+		(property "Value" "Thonkicon"
 			(at 34.29 99.6949 0)
 			(effects
@@
 			)
 		)
-		(property "Value" "~"
+		(property "Value" "Thonkicon"
 			(at 265.43 76.8349 0)
 			(effects
@@
 			)
 		)
-		(property "Value" "~"
+		(property "Value" "Thonkicon"
 			(at 265.43 145.4149 0)
 			(effects
@@
 			)
 		)
-		(property "Value" "~"
+		(property "Value" "Thonkicon"
 			(at 34.29 142.8749 0)
 			(effects
@@
 			)
 		)
-		(property "Value" "~"
+		(property "Value" "Thonkicon"
 			(at 265.43 112.3949 0)
 			(effects
@@
 			)
 		)
-		(property "Value" "~"
+		(property "Value" "Thonkicon"
 			(at 34.29 55.2449 0)
 			(effects
@@
 			)
 		)
-		(property "Value" "LED_Dual_Bidirectional"
+		(property "Value" "Bipolar LED"
 			(at 259.8547 124.46 0)
 			(effects
@@
 			)
 		)
-		(property "Value" "100K"
+		(property "Value" "A100K"
 			(at 39.37 80.01 90)
 			(effects
@@
 			)
 		)
-		(property "Value" "~"
+		(property "Value" "Thonkicon"
 			(at 34.29 188.5949 0)
 			(effects
@@
 			)
 		)
-		(property "Value" "~"
+		(property "Value" "Subminiture SPDT"
 			(at 86.7922 26.797 90)
 			(effects
@@
 			)
 		)
-		(property "Value" "100K"
+		(property "Value" "A100K"
 			(at 39.37 168.91 90)
 			(effects
@@
 			)
 		)
-		(property "Value" "100K"
+		(property "Value" "A100K"
 			(at 39.37 35.56 90)
 			(effects
@@
 			)
 		)
-		(property "Value" "~"
+		(property "Value" "Subminiture SPDT"
 			(at 86.7922 160.147 90)
 			(effects
@@
 			)
 		)
-		(property "Value" "~"
+		(property "Value" "Subminiture SPDT"
 			(at 86.7922 69.977 90)
 			(effects
@@
 			)
 		)
-		(property "Value" "Conn_01x13_Socket"
+		(property "Value" "01x13 Male Pin Header"
 			(at 134.874 35.56 0)
 			(effects
@@
 			)
 		)
-		(property "Value" "~"
+		(property "Value" "Thonkicon"
 			(at 34.29 158.1149 0)
 			(effects
@@
 			)
 		)
-		(property "Value" "Conn_01x09_Socket"
+		(property "Value" "01x09 Male Pin Header"
 			(at 195.58 49.5299 0)
 			(effects
@@
 			)
 		)
-		(property "Value" "100K"
+		(property "Value" "A100K"
 			(at 39.37 124.46 90)
 			(effects
@@
 			)
 		)
-		(property "Value" "~"
+		(property "Value" "Subminiture SPDT"
 			(at 86.7922 114.427 90)
 			(effects
@@
 			)
 		)
-		(property "Value" "~"
+		(property "Value" "Thonkicon"
 			(at 34.29 24.7649 0)
 			(effects
