File: hardware/bottom-board/bottom-board.kicad_pcb (KiCad board)
At the start: 2 copper layers, 39 x 110 mm, 108 parts, among them J1 Conn_01x15_Socket, J2 Conn_01x15_Pin, J3 VCA_TP, J9 PWR, Q1 2N3904, Q2 2N3906, Q3 2N3904, Q4 2N3906, Q5 2N3904, Q6 2N3906, Q7 2N3904, Q8 2N3906, U1 TL084, U2 NE5517, U3 TL084, U4 NE5517, U5 TL072

Commit message: wip - first pass done
Parts:
- removed C10, C11, C12, C7, C8, C9: 100nF, Capacitor_THT:C_Rect_L4.6mm_W3.0mm_P2.50mm_MKS02_FKP02
- removed J9: PWR, Eurorack Common:Eurorack Power Header (10 pin)
- removed Q5, Q7: 2N3904, Package_TO_SOT_THT:TO-92L_HandSolder
- removed Q6, Q8: 2N3906, Package_TO_SOT_THT:TO-92L_HandSolder
- removed R33, R34, R49, R50, R65, R66: 20K, Resistor_THT:R_Axial_DIN0207_L6.3mm_D2.5mm_P7.62mm_Horizontal
- removed R40, R43, R47, R56, R59, R63: 100K, Resistor_THT:R_Axial_DIN0207_L6.3mm_D2.5mm_P7.62mm_Horizontal
- removed R41, R42, R45, R57, R58, R61: 2K, Resistor_THT:R_Axial_DIN0207_L6.3mm_D2.5mm_P7.62mm_Horizontal
- removed R44, R60: 470R, Resistor_THT:R_Axial_DIN0207_L6.3mm_D2.5mm_P7.62mm_Horizontal
- removed R46, R62: 120K, Resistor_THT:R_Axial_DIN0207_L6.3mm_D2.5mm_P7.62mm_Horizontal
- removed R48, R64: 30K, Resistor_THT:R_Axial_DIN0207_L6.3mm_D2.5mm_P7.62mm_Horizontal
- removed R72, R77, R82, R87: 150R, Resistor_THT:R_Axial_DIN0207_L6.3mm_D2.5mm_P7.62mm_Horizontal
- removed R73, R78, R83, R88: 2M, Resistor_THT:R_Axial_DIN0207_L6.3mm_D2.5mm_P7.62mm_Horizontal
- removed R74, R79, R84, R89: 470K, Resistor_THT:R_Axial_DIN0207_L6.3mm_D2.5mm_P7.62mm_Horizontal
- removed R75, R80, R85, R90: 47K, Resistor_THT:R_Axial_DIN0207_L6.3mm_D2.5mm_P7.62mm_Horizontal
- removed R76, R81, R86, R91: 4.7K, Resistor_THT:R_Axial_DIN0207_L6.3mm_D2.5mm_P7.62mm_Horizontal
- removed RV5, RV7: 2K, Potentiometer_THT:Potentiometer_Bourns_3296W_Vertical
- removed RV6, RV8: 100K, Potentiometer_THT:Potentiometer_Bourns_3296W_Vertical
- removed U3: TL084, Package_SO:Texas_DYY0016A_TSOT-23-16_2x4.2mm_P0.5mm
- removed U4: NE5517, Package_SO:JEITA_SOIC-16_3.9x9.9mm_P1.27mm
- removed U5: TL072, Package_DIP:DIP-8_W7.62mm
- added R19: 2K, Eurorack Common:R_Axial_DIN0207_L6.3mm_D2.5mm_P7.62mm_Horizontal, F.Cu at (39.3, 43.8)
- added R20: 100K, Eurorack Common:R_Axial_DIN0207_L6.3mm_D2.5mm_P7.62mm_Horizontal, F.Cu at (31.9, 65.1)
- added R21: 470R, Eurorack Common:R_Axial_DIN0207_L6.3mm_D2.5mm_P7.62mm_Horizontal, F.Cu at (39.5, 68.5)
- added R22: 2K, Eurorack Common:R_Axial_DIN0207_L6.3mm_D2.5mm_P7.62mm_Horizontal, F.Cu at (31.7, 48.0)
- added R23: 120K, Eurorack Common:R_Axial_DIN0207_L6.3mm_D2.5mm_P7.62mm_Horizontal, F.Cu at (24.3, 86.0)
- C1, C2: footprint Capacitor_THT:CP_Radial_D5.0mm_P2.00mm -> Eurorack Common:C_Radial_D5.0mm_H11.0mm_P2.00mm
- C3, C4, C5, C6: footprint Capacitor_THT:C_Rect_L4.6mm_W3.0mm_P2.50mm_MKS02_FKP02 -> Eurorack Common:C_Disc_D3.4mm_W2.1mm_P2.50mm
- J1: value Conn_01x15_Socket -> Conn_01x10_Socket; footprint Connector_PinHeader_2.54mm:PinHeader_1x15_P2.54mm_Vertical -> Connector_PinSocket_2.54mm:PinSocket_1x10_P2.54mm_Vertical
- J2: value Conn_01x15_Pin -> PWR; footprint Connector_PinHeader_2.54mm:PinHeader_1x15_P2.54mm_Vertical -> Eurorack Common:Eurorack Power Header (10 pin); moved to B.Cu
- J3: value VCA_TP -> Conn_01x10_Pin; footprint Connector_PinHeader_2.54mm:PinHeader_1x04_P2.54mm_Vertical -> Connector_PinSocket_2.54mm:PinSocket_1x10_P2.54mm_Vertical; moved to F.Cu
- Q1, Q2, Q3, Q4: footprint Package_TO_SOT_THT:TO-92L_HandSolder -> Eurorack Common:TO-92_Inline
- R1, R24, R4, R8: footprint Resistor_THT:R_Axial_DIN0207_L6.3mm_D2.5mm_P7.62mm_Horizontal -> Eurorack Common:R_Axial_DIN0207_L6.3mm_D2.5mm_P7.62mm_Horizontal
- R10, R26: value 2K -> 20K; footprint Resistor_THT:R_Axial_DIN0207_L6.3mm_D2.5mm_P7.62mm_Horizontal -> Eurorack Common:R_Axial_DIN0207_L6.3mm_D2.5mm_P7.62mm_Horizontal
- R11, R27: value 100K -> 20K; footprint Resistor_THT:R_Axial_DIN0207_L6.3mm_D2.5mm_P7.62mm_Horizontal -> Eurorack Common:R_Axial_DIN0207_L6.3mm_D2.5mm_P7.62mm_Horizontal
- R12, R28: value 470R -> 150R; footprint Resistor_THT:R_Axial_DIN0207_L6.3mm_D2.5mm_P7.62mm_Horizontal -> Eurorack Common:R_Axial_DIN0207_L6.3mm_D2.5mm_P7.62mm_Horizontal
- R13, R29: value 2K -> 2M; footprint Resistor_THT:R_Axial_DIN0207_L6.3mm_D2.5mm_P7.62mm_Horizontal -> Eurorack Common:R_Axial_DIN0207_L6.3mm_D2.5mm_P7.62mm_Horizontal
- R14, R30: value 120K -> 470K; footprint Resistor_THT:R_Axial_DIN0207_L6.3mm_D2.5mm_P7.62mm_Horizontal -> Eurorack Common:R_Axial_DIN0207_L6.3mm_D2.5mm_P7.62mm_Horizontal
- R15, R31: value 100K -> 47K; footprint Resistor_THT:R_Axial_DIN0207_L6.3mm_D2.5mm_P7.62mm_Horizontal -> Eurorack Common:R_Axial_DIN0207_L6.3mm_D2.5mm_P7.62mm_Horizontal
- R16, R32: value 30K -> 4.7K; footprint Resistor_THT:R_Axial_DIN0207_L6.3mm_D2.5mm_P7.62mm_Horizontal -> Eurorack Common:R_Axial_DIN0207_L6.3mm_D2.5mm_P7.62mm_Horizontal
- R17: value 20K -> 100K; footprint Resistor_THT:R_Axial_DIN0207_L6.3mm_D2.5mm_P7.62mm_Horizontal -> Eurorack Common:R_Axial_DIN0207_L6.3mm_D2.5mm_P7.62mm_Horizontal
- R18: value 20K -> 2K; footprint Resistor_THT:R_Axial_DIN0207_L6.3mm_D2.5mm_P7.62mm_Horizontal -> Eurorack Common:R_Axial_DIN0207_L6.3mm_D2.5mm_P7.62mm_Horizontal
- R2, R3, R6: value 100K -> 2K; footprint Resistor_THT:R_Axial_DIN0207_L6.3mm_D2.5mm_P7.62mm_Horizontal -> Eurorack Common:R_Axial_DIN0207_L6.3mm_D2.5mm_P7.62mm_Horizontal
- R25, R9: value 2K -> 30K; footprint Resistor_THT:R_Axial_DIN0207_L6.3mm_D2.5mm_P7.62mm_Horizontal -> Eurorack Common:R_Axial_DIN0207_L6.3mm_D2.5mm_P7.62mm_Horizontal
- R5: value 100K -> 470R; footprint Resistor_THT:R_Axial_DIN0207_L6.3mm_D2.5mm_P7.62mm_Horizontal -> Eurorack Common:R_Axial_DIN0207_L6.3mm_D2.5mm_P7.62mm_Horizontal
- R7: value 100K -> 120K; footprint Resistor_THT:R_Axial_DIN0207_L6.3mm_D2.5mm_P7.62mm_Horizontal -> Eurorack Common:R_Axial_DIN0207_L6.3mm_D2.5mm_P7.62mm_Horizontal
- RV1, RV2, RV3, RV4: footprint Potentiometer_THT:Potentiometer_Bourns_3296W_Vertical -> Eurorack Common:Potentiometer_Bourns_3296W_Horizontal
- U1: footprint Package_SO:Texas_DYY0016A_TSOT-23-16_2x4.2mm_P0.5mm -> Eurorack Common:Texas_DYY0014A_TSOT-23-14_2x4.2mm_P0.5mm
- U2: footprint Package_SO:JEITA_SOIC-16_3.9x9.9mm_P1.27mm -> Eurorack Common:SOIC-16_3.9x9.9mm_P1.27mm
- moved C3 114.9 mm to (40.0, 101.2), turned to 180 degrees
- moved C4 99.5 mm to (40.0, 88.2), turned to 180 degrees
- moved R7 93.4 mm to (31.7, 24.0)
- moved R4 73.9 mm to (31.7, 33.9), turned to 0 degrees
- moved R5 73.7 mm to (39.3, 37.2), turned to 180 degrees
- moved C5 72.5 mm to (37.2, 55.6), turned to 180 degrees
- moved R32 71.6 mm to (34.8, 107.6), turned to 0 degrees
- moved R25 68.9 mm to (24.3, 93.5)
- moved R16 67.8 mm to (34.8, 104.6), turned to 0 degrees
- moved R26 66.8 mm to (31.9, 97.2), turned to 180 degrees
- moved R24 65.2 mm to (24.3, 89.8)
- moved C6 65.1 mm to (37.2, 48.0), turned to 180 degrees
- moved R6 59.0 mm to (40.0, 55.6), turned to 90 degrees
- moved R3 56.1 mm to (31.9, 61.8)
- moved U2 55.6 mm to (39.0, 94.8)
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Connections:
- J1 pad 1: -12V -> +12V
- J1 pad 10: /IN_B -> -12V
- J1 pad 2: /OFFSET_A -> GND
- J1 pad 3: /IN_A -> /OFFSET_C
- J1 pad 4: /MIX_A -> /IN_C
- J1 pad 5: /OUT_A -> /OUT_C
- J1 pad 6: /LIN_A -> /LIN_C
- J1 pad 7: /LOG_A -> /LOG_C
- J1 pad 8: /COMMON_A -> /COMMON_C
- J1 pad 9: /OFFSET_B -> GND
- J2 pad 1: GND -> -12V
- J2 pad 10: /OFFSET_D -> +12V
- J2 pad 2: +12V -> -12V
- J2 pad 3: /OFFSET_C -> GND
- J2 pad 4: /IN_C -> GND
- J2 pad 5: /MIX_C -> GND
- J2 pad 6: /OUT_C -> GND
- J2 pad 7: /LIN_C -> GND
- J2 pad 8: /LOG_C -> GND
- J2 pad 9: /COMMON_C -> +12V
- J3 pad 1: /OUT_A -> +12V
- J3 pad 2: /OUT_B -> GND
- J3 pad 3: /OUT_C -> /OFFSET_D
- J3 pad 4: /OUT_D -> /IN_D
- R1 pad 1: /MIX_A -> +12V
- R1 pad 2: Net-(U5A--) -> Net-(U1A-+)
- R10 pad 1: /OFFSET_A -> /LIN_C
- R10 pad 2: Net-(Q1-B) -> -12V
- R11 pad 1: Net-(U1B-+) -> Net-(Q2-C)
- R11 pad 2: +12V -> /LOG_C
- R12 pad 1: GND -> Net-(R12-Pad1)
- R12 pad 2: Net-(U1B-+) -> GND
- R13 pad 1: Net-(Q1-B) -> /VCA_C/BIAS
- R13 pad 2: Net-(U1B--) -> Net-(R13-Pad2)
- R14 pad 1: -12V -> Net-(R13-Pad2)
- R14 pad 2: Net-(Q1-E) -> +12V
- R15 pad 1: Net-(R15-Pad1) -> GND
- R15 pad 2: Net-(U1B--) -> Net-(R13-Pad2)
- R16 pad 1: Net-(R15-Pad1) -> -12V
- R16 pad 2: /LIN_A -> /OUT_C
- R17 pad 1: /LIN_A -> +12V
- R17 pad 2: -12V -> Net-(U1C-+)
- R18 pad 1: Net-(Q2-C) -> Net-(U1C-+)
- R18 pad 2: /LOG_A -> GND
- R2 pad 1: /MIX_B -> Net-(U1A-+)
- R2 pad 2: Net-(U5A--) -> GND
- R24 pad 1: +12V -> Net-(R24-Pad1)
- R24 pad 2: Net-(U1C-+) -> Net-(U1D--)
- R25 pad 1: Net-(U1C-+) -> Net-(R24-Pad1)
- R25 pad 2: GND -> /LIN_D
- R26 pad 1: /OFFSET_B -> /LIN_D
- R26 pad 2: Net-(Q3-B) -> -12V
- R27 pad 1: Net-(U1D-+) -> Net-(Q4-C)
- R27 pad 2: +12V -> /LOG_D
- R28 pad 1: GND -> Net-(R28-Pad1)
- R28 pad 2: Net-(U1D-+) -> GND
- R29 pad 1: Net-(Q3-B) -> /VCA_D/BIAS
- R29 pad 2: Net-(U1D--) -> Net-(R29-Pad2)
- R3 pad 1: /MIX_C -> /OFFSET_C
- R3 pad 2: Net-(U5A--) -> Net-(Q1-B)
- R30 pad 1: -12V -> Net-(R29-Pad2)
- R30 pad 2: Net-(Q3-E) -> +12V
- R31 pad 1: Net-(R31-Pad1) -> GND
- R31 pad 2: Net-(U1D--) -> Net-(R29-Pad2)
- R32 pad 1: Net-(R31-Pad1) -> -12V
- R32 pad 2: /LIN_B -> /OUT_D
- R4 pad 1: /OUT_D -> Net-(U1B-+)
- R4 pad 2: Net-(U5A--) -> +12V
- R5 pad 1: Net-(U5A--) -> GND
- R5 pad 2: Net-(R5-Pad2) -> Net-(U1B-+)
- R6 pad 1: Net-(R5-Pad2) -> Net-(Q1-B)
- R6 pad 2: Net-(U5B--) -> Net-(U1B--)
- R7 pad 1: Net-(U5B--) -> -12V
- R7 pad 2: /MIX_OUT -> Net-(Q1-E)
- R8 pad 1: +12V -> Net-(R8-Pad1)
- R8 pad 2: Net-(U1A-+) -> Net-(U1B--)
- R9 pad 1: Net-(U1A-+) -> Net-(R8-Pad1)
- R9 pad 2: GND -> /LIN_C
- RV1 pad 1: /IN_A -> /IN_C
- RV1 pad 2: /IN_A -> /IN_C
- RV1 pad 3: Net-(R72-Pad1) -> Net-(R12-Pad1)
- RV2 pad 2: /VCA_A/BIAS -> /VCA_C/BIAS
- RV3 pad 1: /IN_B -> /IN_D
- RV3 pad 2: /IN_B -> /IN_D
- RV3 pad 3: Net-(R77-Pad1) -> Net-(R28-Pad1)
- RV4 pad 2: /VCA_B/BIAS -> /VCA_D/BIAS
- U1 pad 14: Net-(R31-Pad1) -> Net-(R24-Pad1)
- U1 pad 2: /OFFSET_A -> /OFFSET_C
- U1 pad 7: Net-(R15-Pad1) -> Net-(R8-Pad1)
- U1 pad 9: /OFFSET_B -> /OFFSET_D
- U2 pad 1: /COMMON_A -> /COMMON_D
- U2 pad 10: Net-(R78-Pad2) -> Net-(R13-Pad2)
- U2 pad 12: Net-(R78-Pad2) -> Net-(R13-Pad2)
- U2 pad 14: /IN_B -> /IN_C
- U2 pad 16: /COMMON_B -> /COMMON_C
- U2 pad 3: /IN_A -> /IN_D
- U2 pad 5: Net-(R73-Pad2) -> Net-(R29-Pad2)
- U2 pad 7: Net-(R73-Pad2) -> Net-(R29-Pad2)
- U2 pad 8: /OUT_A -> /OUT_D
- U2 pad 9: /OUT_B -> /OUT_C
Routing:
- net +12V: track 150.1 -> 28.3 mm, vias 7 -> 3
- net /MIX_B: track 108.1 -> 0.00 mm, vias 1 -> 0
- net /IN_D: track 0.00 -> 102.4 mm, vias 0 -> 3
- net /OFFSET_D: track 0.00 -> 97.0 mm, vias 0 -> 3
- net /MIX_A: track 92.1 -> 0.00 mm
- net /OUT_C: track 0.00 -> 80.9 mm, vias 0 -> 2
- net /IN_C: track 0.00 -> 75.6 mm, vias 0 -> 1
- net /COMMON_C: track 0.00 -> 74.6 mm, vias 0 -> 3
- net Net-(R29-Pad2): track 0.00 -> 72.2 mm, vias 0 -> 2
- net -12V: track 115.1 -> 50.8 mm, vias 4 -> 3
- net Net-(Q3-B): track 7.68 -> 59.8 mm
- net Net-(R24-Pad1): track 0.00 -> 49.4 mm, vias 0 -> 1
- net Net-(R13-Pad2): track 0.00 -> 42.5 mm, vias 0 -> 2
- net /LIN_D: track 0.00 -> 41.8 mm, vias 0 -> 1
- net /OFFSET_C: track 0.00 -> 37.7 mm, vias 0 -> 3
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- added copper zone on In2.Cu, net +12V
- added copper zone on In2.Cu, net -12V
- added copper zone on In1.Cu, net GND
Other:
- copper layers 2 -> 4
- board text added: "BIAS C"
- board text added: "BIAS D"
- board text added: "Q-VCA-M v1"
- board text added: "TRIM C"
- board text added: "TRIM D"

Commit message: chore: clean up the boards
Parts:
- J1: value Conn_01x10_Socket -> 01x10 Female Pin Header
- J3: value Conn_01x10_Pin -> 01x10 Female Pin Header
- RV2, RV4: value 100K -> B100K
