File: hardware/bottom-board/bottom-board.kicad_sch (KiCad schematic)
At the start: 11 parts, among them J1 Conn_01x15_Socket, J2 PWR, J3 Conn_01x13_Pin, U1 TL084, U2 NE5517

Commit message: wip - first pass done
Parts:
- C1, C2: footprint Capacitor_THT:CP_Radial_D5.0mm_P2.00mm -> Eurorack Common:C_Radial_D5.0mm_H11.0mm_P2.00mm; symbol Device:C_Polarized -> Eurorack Common:CP_ESH_10uF_50V_Radial_D5_L11
- C3, C4, C5, C6: footprint Capacitor_THT:C_Rect_L4.6mm_W3.0mm_P2.50mm_MKS02_FKP02 -> Eurorack Common:C_Disc_D3.4mm_W2.1mm_P2.50mm; symbol Device:C -> Eurorack Common:C_100nF_50V_X7R_2.5mm
- J1: value Conn_01x15_Socket -> Conn_01x10_Socket; footprint Connector_PinHeader_2.54mm:PinHeader_1x15_P2.54mm_Vertical -> Connector_PinSocket_2.54mm:PinSocket_1x10_P2.54mm_Vertical
- J2: symbol Connector_Generic:Conn_02x05_Odd_Even -> Eurorack Common:Eurorack_Power_Header_(10_pin)
- J3: value Conn_01x13_Pin -> Conn_01x10_Pin; footprint Connector_PinHeader_2.54mm:PinHeader_1x13_P2.54mm_Vertical -> Connector_PinSocket_2.54mm:PinSocket_1x10_P2.54mm_Vertical
- U1: footprint Package_SO:Texas_DYY0016A_TSOT-23-16_2x4.2mm_P0.5mm -> Eurorack Common:Texas_DYY0014A_TSOT-23-14_2x4.2mm_P0.5mm; symbol Amplifier_Operational:TL084 -> Eurorack Common:TL084HIDYYR
- U2: footprint Package_SO:JEITA_SOIC-16_3.9x9.9mm_P1.27mm -> Eurorack Common:SOIC-16_3.9x9.9mm_P1.27mm; symbol Amplifier_Operational:LM13700 -> Eurorack Common:NE5517DR2G
Changed lines of the file:
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@@
 	)
 	(symbol
-		(lib_id "Device:C")
+		(lib_id "Eurorack Common:C_100nF_50V_X7R_2.5mm")
 		(at 52.07 130.81 0)
 		(unit 1)
@@
 		(fields_autoplaced yes)
 		(property "Reference" "C3"
-			(at 54.991 129.9753 0)
+			(at 55.88 129.5399 0)
 			(effects
 				(font
@@
 		)
 		(property "Value" "100nF"
-			(at 54.991 132.5122 0)
+			(at 55.88 132.0799 0)
 			(effects
 				(font
@@
 			)
 		)
-		(property "Footprint" "Capacitor_THT:C_Rect_L4.6mm_W3.0mm_P2.50mm_MKS02_FKP02"
+		(property "Footprint" "Eurorack Common:C_Disc_D3.4mm_W2.1mm_P2.50mm"
 			(at 53.0352 134.62 0)
 			(effects
@@
 			)
 		)
-		(property "Description" ""
+		(property "Description" "Unpolarized capacitor"
 			(at 52.07 130.81 0)
 			(effects
@@
 					(size 1.27 1.27)
 				)
+				(hide yes)
 			)
 		)
@@
 	)
 	(symbol
-		(lib_id "Amplifier_Operational:TL084")
+		(lib_id "Eurorack Common:TL084HIDYYR")
 		(at 48.26 135.89 0)
 		(unit 5)
@@
 		(fields_autoplaced yes)
 		(property "Reference" "U1"
-			(at 46.355 135.0553 0)
+			(at 46.99 134.6199 0)
 			(effects
 				(font
@@
 		)
 		(property "Value" "TL084"
-			(at 46.355 137.5922 0)
+			(at 46.99 137.1599 0)
 			(effects
 				(font
@@
 			)
 		)
-		(property "Footprint" "Package_SO:Texas_DYY0016A_TSOT-23-16_2x4.2mm_P0.5mm"
+		(property "Footprint" "Eurorack Common:Texas_DYY0014A_TSOT-23-14_2x4.2mm_P0.5mm"
 			(at 46.99 133.35 0)
 			(effects
@@
 			)
 		)
-		(property "Datasheet" "http://www.ti.com/lit/ds/symlink/tl081.pdf"
+		(property "Datasheet" "http://www.ti.com/lit/ds/symlink/tl084.pdf"
 			(at 49.53 130.81 0)
 			(effects
@@
 			)
 		)
-		(property "Description" ""
+		(property "Description" "Low-Power, Quad-Operational Amplifiers, TSOT-23-14"
 			(at 48.26 135.89 0)
 			(effects
@@
 					(size 1.27 1.27)
 				)
+				(hide yes)
 			)
 		)
@@
 	)
 	(symbol
-		(lib_id "Device:C")
+		(lib_id "Eurorack Common:C_100nF_50V_X7R_2.5mm")
 		(at 52.07 140.97 0)
 		(unit 1)
@@
 		(fields_autoplaced yes)
 		(property "Reference" "C4"
-			(at 54.991 140.1353 0)
+			(at 55.88 139.6999 0)
 			(effects
 				(font
@@
 		)
 		(property "Value" "100nF"
-			(at 54.991 142.6722 0)
+			(at 55.88 142.2399 0)
 			(effects
 				(font
@@
 			)
 		)
-		(property "Footprint" "Capacitor_THT:C_Rect_L4.6mm_W3.0mm_P2.50mm_MKS02_FKP02"
+		(property "Footprint" "Eurorack Common:C_Disc_D3.4mm_W2.1mm_P2.50mm"
 			(at 53.0352 144.78 0)
 			(effects
@@
 			)
 		)
-		(property "Description" ""
+		(property "Description" "Unpolarized capacitor"
 			(at 52.07 140.97 0)
 			(effects
@@
 					(size 1.27 1.27)
 				)
+				(hide yes)
 			)
 		)
@@
 	)
 	(symbol
-		(lib_id "Device:C")
+		(lib_id "Eurorack Common:C_100nF_50V_X7R_2.5mm")
 		(at 74.93 130.81 0)
 		(unit 1)
@@
 		(fields_autoplaced yes)
 		(property "Reference" "C5"
-			(at 77.851 129.9753 0)
+			(at 78.74 129.5399 0)
 			(effects
 				(font
@@
 		)
 		(property "Value" "100nF"
-			(at 77.851 132.5122 0)
+			(at 78.74 132.0799 0)
 			(effects
 				(font
@@
 			)
 		)
-		(property "Footprint" "Capacitor_THT:C_Rect_L4.6mm_W3.0mm_P2.50mm_MKS02_FKP02"
+		(property "Footprint" "Eurorack Common:C_Disc_D3.4mm_W2.1mm_P2.50mm"
 			(at 75.8952 134.62 0)
 			(effects
@@
 			)
 		)
-		(property "Description" ""
+		(property "Description" "Unpolarized capacitor"
 			(at 74.93 130.81 0)
 			(effects
@@
 					(size 1.27 1.27)
 				)
+				(hide yes)
 			)
 		)
@@
 			)
 		)
-		(property "Value" "Conn_01x15_Socket"
+		(property "Value" "Conn_01x10_Socket"
 			(at 20.574 27.94 0)
 			(effects
@@
 			)
 		)
-		(property "Footprint" "Connector_PinHeader_2.54mm:PinHeader_1x15_P2.54mm_Vertical"
+		(property "Footprint" "Connector_PinSocket_2.54mm:PinSocket_1x10_P2.54mm_Vertical"
 			(at 35.56 40.64 0)
 			(effects
@@
 	)
 	(symbol
-		(lib_id "Connector_Generic:Conn_02x05_Odd_Even")
+		(lib_id "Eurorack Common:Eurorack_Power_Header_(10_pin)")
 		(at 40.64 93.98 0)
 		(unit 1)
@@
 			)
 		)
-		(property "Value" "Conn_01x13_Pin"
+		(property "Value" "Conn_01x10_Pin"
 			(at 52.07 27.178 0)
 			(effects
@@
 			)
 		)
-		(property "Footprint" "Connector_PinHeader_2.54mm:PinHeader_1x13_P2.54mm_Vertical"
+		(property "Footprint" "Connector_PinSocket_2.54mm:PinSocket_1x10_P2.54mm_Vertical"
 			(at 57.15 40.64 0)
 			(effects
@@
 	)
 	(symbol
-		(lib_id "Device:C_Polarized")
+		(lib_id "Eurorack Common:CP_ESH_10uF_50V_Radial_D5_L11")
 		(at 30.48 140.97 0)
 		(unit 1)
@@
 		(fields_autoplaced yes)
 		(property "Reference" "C2"
-			(at 33.401 139.2463 0)
+			(at 34.29 138.8109 0)
 			(effects
 				(font
@@
 		)
 		(property "Value" "10uF"
-			(at 33.401 141.7832 0)
+			(at 34.29 141.3509 0)
 			(effects
 				(font
@@
 			)
 		)
-		(property "Footprint" "Capacitor_THT:CP_Radial_D5.0mm_P2.00mm"
+		(property "Footprint" "Eurorack Common:C_Radial_D5.0mm_H11.0mm_P2.00mm"
 			(at 31.4452 144.78 0)
 			(effects
@@
 			)
 		)
-		(property "Description" ""
+		(property "Description" "Polarized capacitor"
 			(at 30.48 140.97 0)
 			(effects
@@
 					(size 1.27 1.27)
 				)
+				(hide yes)
 			)
 		)
@@
 	)
 	(symbol
-		(lib_id "Device:C")
+		(lib_id "Eurorack Common:C_100nF_50V_X7R_2.5mm")
 		(at 74.93 140.97 0)
 		(unit 1)
@@
 		(fields_autoplaced yes)
 		(property "Reference" "C6"
-			(at 77.851 140.1353 0)
+			(at 78.74 139.6999 0)
 			(effects
 				(font
@@
 		)
 		(property "Value" "100nF"
-			(at 77.851 142.6722 0)
+			(at 78.74 142.2399 0)
 			(effects
 				(font
@@
 			)
 		)
-		(property "Footprint" "Capacitor_THT:C_Rect_L4.6mm_W3.0mm_P2.50mm_MKS02_FKP02"
+		(property "Footprint" "Eurorack Common:C_Disc_D3.4mm_W2.1mm_P2.50mm"
 			(at 75.8952 144.78 0)
 			(effects
@@
 			)
 		)
-		(property "Description" ""
+		(property "Description" "Unpolarized capacitor"
 			(at 74.93 140.97 0)
 			(effects
@@
 					(size 1.27 1.27)
 				)
+				(hide yes)
 			)
 		)
@@
 	)
 	(symbol
-		(lib_id "Amplifier_Operational:LM13700")
+		(lib_id "Eurorack Common:NE5517DR2G")
 		(at 68.58 135.89 0)
 		(unit 5)
@@
 			)
 		)
-		(property "Footprint" "Package_SO:JEITA_SOIC-16_3.9x9.9mm_P1.27mm"
+		(property "Footprint" "Eurorack Common:SOIC-16_3.9x9.9mm_P1.27mm"
 			(at 60.96 135.255 0)
 			(effects
@@
 			)
 		)
-		(property "Datasheet" ""
+		(property "Datasheet" "https://www.onsemi.com/download/data-sheet/pdf/ne5517-d.pdf"
 			(at 60.96 135.255 0)
 			(effects
@@
 			)
 		)
-		(property "Description" ""
+		(property "Description" "Dual Operational Transconductance Amplifiers with Linearizing Diodes and Buffers, SOIC-16, drop in replacement for LM13700"
 			(at 68.58 135.89 0)
 			(effects
@@
 	)
 	(symbol
-		(lib_id "Device:C_Polarized")
+		(lib_id "Eurorack Common:CP_ESH_10uF_50V_Radial_D5_L11")
 		(at 30.48 130.81 0)
 		(unit 1)
@@
 		(fields_autoplaced yes)
 		(property "Reference" "C1"
-			(at 33.401 129.0863 0)
+			(at 34.29 128.6509 0)
 			(effects
 				(font
@@
 		)
 		(property "Value" "10uF"
-			(at 33.401 131.6232 0)
+			(at 34.29 131.1909 0)
 			(effects
 				(font
@@
 			)
 		)
-		(property "Footprint" "Capacitor_THT:CP_Radial_D5.0mm_P2.00mm"
+		(property "Footprint" "Eurorack Common:C_Radial_D5.0mm_H11.0mm_P2.00mm"
 			(at 31.4452 134.62 0)
 			(effects
@@
 			)
 		)
-		(property "Description" ""
+		(property "Description" "Polarized capacitor"
 			(at 30.48 130.81 0)
 			(effects
@@
 					(size 1.27 1.27)
 				)
-			)
-		)
+				(hide yes)
+			)
+		)

Commit message: chore: clean up the boards
Parts:
- J1: value Conn_01x10_Socket -> 01x10 Female Pin Header
- J3: value Conn_01x10_Pin -> 01x10 Female Pin Header
Changed lines of the file:
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@@
 			)
 		)
-		(property "Value" "Conn_01x10_Socket"
+		(property "Value" "01x10 Female Pin Header"
 			(at 20.574 27.94 0)
 			(effects
@@
 			)
 		)
-		(property "Value" "Conn_01x10_Pin"
+		(property "Value" "01x10 Female Pin Header"
 			(at 52.07 27.178 0)
 			(effects

Commit message: chore: add description and data sheet to ibom
Parts:
- C1, C2: Notes (none) -> Bulk decoupling
Changed lines of the file:
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@@
+			)
+		)
+		(property "Notes" ""
+			(at 52.07 130.81 0)
+			(effects
+				(font
+					(size 1.27 1.27)
+				)
+				(hide yes)
 			)
 		)
@@
 			)
 		)
+		(property "Notes" ""
+			(at 48.26 135.89 0)
+			(effects
+				(font
+					(size 1.27 1.27)
+				)
+				(hide yes)
+			)
+		)
 		(pin "1"
 		)
@@
 			)
 		)
+		(property "Notes" ""
+			(at 52.07 140.97 0)
+			(effects
+				(font
+					(size 1.27 1.27)
+				)
+				(hide yes)
+			)
+		)
 		(pin "1"
 		)
@@
 			)
 		)
+		(property "Notes" ""
+			(at 74.93 130.81 0)
+			(effects
+				(font
+					(size 1.27 1.27)
+				)
+				(hide yes)
+			)
+		)
 		(pin "1"
 		)
@@
 		)
 		(property "Description" "Generic connector, single row, 01x10, script generated"
+			(at 35.56 40.64 0)
+			(effects
+				(font
+					(size 1.27 1.27)
+				)
+				(hide yes)
+			)
+		)
+		(property "Notes" ""
 			(at 35.56 40.64 0)
 			(effects
@@
 			)
 		)
+		(property "Notes" ""
+			(at 40.64 93.98 0)
+			(effects
+				(font
+					(size 1.27 1.27)
+				)
+				(hide yes)
+			)
+		)
 		(pin "1"
 		)
@@
 		)
 		(property "Description" "Generic connector, single row, 01x10, script generated"
+			(at 57.15 40.64 0)
+			(effects
+				(font
+					(size 1.27 1.27)
+				)
+				(hide yes)
+			)
+		)
+		(property "Notes" ""
 			(at 57.15 40.64 0)
 			(effects
@@
 			)
 		)
+		(property "Notes" "Bulk decoupling"
+			(at 30.48 140.97 0)
+			(effects
+				(font
+					(size 1.27 1.27)
+				)
+				(hide yes)
+			)
+		)
 		(pin "1"
 		)
@@
 			)
 		)
+		(property "Notes" ""
+			(at 74.93 140.97 0)
+			(effects
+				(font
+					(size 1.27 1.27)
+				)
+				(hide yes)
+			)
+		)
 		(pin "1"
 		)
@@
 			)
 		)
+		(property "Notes" ""
+			(at 68.58 135.89 0)
+			(effects
+				(font
+					(size 1.27 1.27)
+				)
+				(hide yes)
+			)
+		)
 		(pin "3"
 		)
@@
 			(at 30.48 130.81 0)
 			(effects
+				(font
+					(size 1.27 1.27)
+				)
+				(hide yes)
+			)
+		)
+		(property "Notes" "Bulk decoupling"
+			(at 30.48 130.81 0)
+			(effects

Commit message: fix: inverted power pins on op amps
Parts:
- C1, C2: footprint Eurorack Common:C_Radial_D5.0mm_H11.0mm_P2.00mm -> Eurorack Common:CP_Radial_D5.0mm_H11.0mm_P2.00mm
Changed lines of the file:
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@@
 			)
 		)
-		(property "Footprint" "Eurorack Common:C_Radial_D5.0mm_H11.0mm_P2.00mm"
+		(property "Footprint" "Eurorack Common:CP_Radial_D5.0mm_H11.0mm_P2.00mm"
 			(at 31.4452 144.78 0)
 			(effects
@@
 			)
 		)
-		(property "Footprint" "Eurorack Common:C_Radial_D5.0mm_H11.0mm_P2.00mm"
+		(property "Footprint" "Eurorack Common:CP_Radial_D5.0mm_H11.0mm_P2.00mm"
 			(at 31.4452 134.62 0)
 			(effects
