File: hardware/front-panel/front-panel.kicad_pcb (KiCad board)
At the start: 2 copper layers, 40.4 x 128.5 mm, 45 parts, among them J1 Thonkicon, J13 Thonkicon, J14 Thonkicon, J15 Thonkicon, J16 Thonkicon, J2 Thonkicon, J3 Thonkicon, J4 Thonkicon, J5 Thonkicon, J6 Thonkicon, J7 Thonkicon, J8 Thonkicon, SW1 Subminiture SPDT, SW2 Subminiture SPDT, SW3 Subminiture SPDT, SW4 Subminiture SPDT

Commit message: feature: docs
Changed lines of the file:
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@@
 		(allow_soldermask_bridges_in_footprints no)
 		(tenting front back)
-		(grid_origin 25.42 25.4)
+		(grid_origin 56.875911 131.211708)
 		(pcbplotparams
 			(layerselection 0x00000000_00000000_55555555_5755f5ff)
@@
 	(gr_poly
 		(pts
-			(xy 64.7 92.929302) (xy 53.8 92.929302) (xy 53.8 104.729302) (xy 60 104.729302) (xy 64.7 100.029302)
+			(xy 64.7 92.929302) (xy 53.8 92.929302) (xy 53.8 104.729302) (xy 55.4 104.729302) (xy 56.9 104.729302)
+			(xy 60 104.729302) (xy 64.7 100.029302)
 		)
 		(stroke
