File: hardware/front-panel/front-panel.kicad_sch (KiCad schematic)
At the start: 28 parts, among them J1 Thonkicon, J13 Thonkicon, J14 Thonkicon, J15 Thonkicon, J16 Thonkicon, J2 Thonkicon, J3 Thonkicon, J4 Thonkicon, J5 Thonkicon, J6 Thonkicon, J7 Thonkicon, J8 Thonkicon, SW1 Subminiture SPDT, SW2 Subminiture SPDT, SW3 Subminiture SPDT, SW4 Subminiture SPDT

Commit message: feature: docs
Connections:
- no-connect marks 68 -> 70
Changed lines of the file:
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@@
+	)
+	(no_connect
+		(at 100.33 179.07)
 	)
 	(no_connect
@@
 	)
 	(no_connect
+		(at 100.33 185.42)
+	)
+	(no_connect
